File: MacroPad.kicad_sch (KiCad schematic)
At the start: 0 parts

Commit message: setting libraries
Other:
- title: (none) -> MacroPad
Changed lines of the file:
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@@
 	(generator_version "9.0")
 	(paper "A4")
+	(title_block
+		(title "MacroPad")
+		(date "2025-05-19")
+		(rev "0")
+	)
 	(sheet_instances
 		(path "/"

Commit message: schematic completed
Parts:
- added D1, D10, D11, D12, D13, D14, D15, D16, D2, D3, D4, D5, D6, D7, D8, D9: Diode, ScottoKeebs_Components:Diode_DO-35, symbol Scottokeebs:Placeholder_Diode
- added S1, S10, S11, S12, S13, S14, S15, S16, S2, S3, S4, S5, S6, S7, S8, S9: Keyswitch, ScottoKeebs_MX:MX_PCB_1.00u, symbol Scottokeebs:Placeholder_Keyswitch
- added SW1: RotaryEncoder_Switch_1, symbol Device:RotaryEncoder_Switch
- added SW2: RotaryEncoder_Switch_2, symbol Device:RotaryEncoder_Switch
- added SW3: RotaryEncoder_Switch_3, symbol Device:RotaryEncoder_Switch
- added U1: ESP32-DevKitC, PCM_Espressif:ESP32-DevKitC, symbol PCM_Espressif:ESP32-DevKitC
Connections:
- new net: D6.2 (A), S6.2
- new net: D3.2 (A), S3.2
- new net: D10.2 (A), S10.2
- new net: D12.2 (A), S12.2
- new net: D8.2 (A), S8.2
- new net: D14.2 (A), S14.2
- new net: D7.2 (A), S7.2
- new net: D16.2 (A), S16.2
- new net: D1.2 (A), S1.2
- new net: D13.2 (A), S13.2
- new net: D15.2 (A), S15.2
- new net: D9.2 (A), S9.2
- new net: D5.2 (A), S5.2
- new net: D4.2 (A), S4.2
- new net: D2.2 (A), S2.2
- new net: D11.2 (A), S11.2
- new net Column 0: S1.1, S13.1, S4.1, S7.1, U1.27 (GPIO16)
- new net Column 1: S14.1, S2.1, S5.1, S8.1, U1.28 (GPIO17)
- new net Column 2: S15.1, S3.1, S6.1, S9.1, U1.30 (GPIO18)
- new net Column 3: S10.1, S11.1, S12.1, S16.1, U1.31 (GPIO19)
- new net Encode1_S1: SW1.S1, U1.11 (ADC2_CH7/GPIO27)
- new net Encode2_S1: SW2.S1, U1.15 (MTCK/GPIO13/ADC2_CH4)
- new net Encode3_S1: SW3.S1, U1.3 (SENSOR_VP/GPIO36/ADC1_CH0)
- new net Encoder1_A: SW1.A, U1.7 (32K_XP/GPIO32/ADC1_CH4)
- new net Encoder1_B: SW1.B, U1.8 (32K_XN/GPIO33/ADC1_CH5)
- new net Encoder2_A: SW2.A, U1.10 (DAC_2/ADC2_CH9/GPIO26)
- new net Encoder2_B: SW2.B, U1.12 (MTMS/GPIO14/ADC2_CH6)
- new net Encoder3_A: SW3.A, U1.26 (ADC2_CH0/GPIO4)
- new net Encoder3_B: SW3.B, U1.29 (GPIO5)
- new net GND: SW1.C, SW1.S2, SW2.C, SW2.S2, SW3.C, SW3.S2, U1.14 (GND), U1.32 (GND), U1.38 (GND)
- new net Row 0: D1.1 (K), D10.1 (K), D2.1 (K), D3.1 (K), U1.33 (GPIO21)
- new net Row 1: D11.1 (K), D4.1 (K), D5.1 (K), D6.1 (K), U1.36 (GPIO22)
- new net Row 2: D12.1 (K), D7.1 (K), D8.1 (K), D9.1 (K), U1.37 (GPIO23)
- new net Row 3: D13.1 (K), D14.1 (K), D15.1 (K), D16.1 (K), U1.9 (DAC_1/ADC2_CH8/GPIO25)
